File: schematics/rep_stm.kicad_pcb (KiCad board)
At the start: 2 copper layers, 122 parts, among them IC1 MOC3011M, IC2 MOC3011M, IC3 MOC3011M, IC4 MOC3011M, P10 THERM1, P11 THERM2, P12 ANALOG IN, P13 END1, P14 END2, P15 END3, P16 END4, P17 DIGITAL INP, P18 USB-MINI-B, P19 PWM 1, P2 BOOT, P20 PWM 2, P21 PWM 3, P22 PWM 4, P3 PROG, P4 DRIVE 1, P5 DRIVE 2, P6 DRIVE 3, P7 DRIVE 4, P8 DRIVE 5, P9 DIGITAL OUT, Q1 BC808-40, Q10 IRF1404S, Q11 BC818-40, Q12 BC808-40, Q13 IRF1404S, Q2 BC818-40, Q3 BC808-40, Q4 IRF1404S, Q5 BC818-40, Q6 BC808-40, Q7 IRF1404S, Q8 BC818-40, Q9 BC808-40, U1 MC34063, U2 STM32F103VE, U3 24C512

Commit message: Start drawing a PCB
Parts:
- added C35: 100n, c_0805, B.Cu at (281.3, 97.8)
- added C36: 100n, c_0805, B.Cu at (281.3, 164.5)
- added C37: 100n, c_0805, B.Cu at (281.3, 75.6)
- added C38: 100n, c_0805, B.Cu at (281.3, 120.0)
- added C39: 100n, c_0805, B.Cu at (281.3, 142.2)
- added U4: POLOLU_A4988, SWDIP8_.6W, F.Cu at (282.6, 146.1)
- added U5: POLOLU_A4988, SWDIP8_.6W, F.Cu at (282.6, 168.3)
- added U6: POLOLU_A4988, SWDIP8_.6W, F.Cu at (282.6, 101.6)
- added U7: POLOLU_A4988, SWDIP8_.6W, F.Cu at (282.6, 123.8)
- added U8: POLOLU_A4988, SWDIP8_.6W, F.Cu at (282.6, 79.4)
- R10, R11, R12, R9: footprint SM0805_Opendous -> SM0805
- moved Q4 219.1 mm to (329.6, 84.5), turned to 0 degrees
- moved P19 218.6 mm to (327.7, 70.5)
- moved Q3 176.7 mm to (323.2, 89.5), turned to 180 degrees
- moved Q7 174.0 mm to (309.2, 84.5), turned to 0 degrees
- moved P20 173.5 mm to (306.7, 70.5)
- moved Q2 169.0 mm to (320.0, 90.8), turned to 180 degrees
- moved R24 167.5 mm to (321.9, 93.3), turned to 90 degrees
- moved IC1 166.1 mm to (324.5, 101.0)
- moved IC2 163.4 mm to (314.3, 101.0)
- moved R25 161.6 mm to (323.9, 93.3), turned to 90 degrees
- moved R26 160.7 mm to (323.2, 86.4)
- moved R28 155.8 mm to (313.7, 93.3), turned to 90 degrees
- moved Q5 154.5 mm to (309.9, 90.8), turned to 180 degrees
- moved R27 153.3 mm to (311.8, 93.3), turned to 90 degrees
- moved Q6 152.0 mm to (313.1, 89.5), turned to 180 degrees
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Connections:
- C18 pad 2: VDD -> +12V
- C19 pad 2: VDD -> +12V
- C20 pad 2: VDD -> +12V
- C21 pad 2: VDD -> +12V
- C22 pad 2: VDD -> +12V
- P19 pad 3: N-0000047 -> N-0000067
- P19 pad 4: N-0000047 -> N-0000067
- P20 pad 3: N-0000044 (its old number) -> N-0000063
- P20 pad 4: N-0000044 (its old number) -> N-0000063
- P21 pad 3: N-0000027 (its old number) -> N-0000013
- P21 pad 4: N-0000027 (its old number) -> N-0000013
- P22 pad 3: N-0000024 (its old number) -> N-0000019
- P22 pad 4: N-0000024 (its old number) -> N-0000019
- Q10 pad 1: N-0000027 (its old number) -> N-0000014
- Q10 pad 2: N-000005 -> N-0000013
- Q13 pad 1: N-0000024 (its old number) -> N-0000021
- Q13 pad 2: N-0000021 -> N-0000019
- Q4 pad 1: N-0000047 -> N-00000152
- Q4 pad 2: N-0000012 -> N-0000067
- Q7 pad 1: N-0000044 (its old number) -> N-00000146
- Q7 pad 2: N-0000017 (its old number) -> N-0000063
- R26 pad 2: N-0000012 -> N-00000152
- R29 pad 2: N-0000017 (its old number) -> N-00000146
- R32 pad 2: N-000005 -> N-0000014
Routing:
- net VCOM: track 22.2 -> 244.7 mm
- net VREF-: track 194.1 -> 36.1 mm, vias 39 -> 3
- net VDD: track 21.6 -> 169.1 mm, vias 5 -> 10
- net VREF+: track 103.2 -> 24.7 mm, vias 2 -> 1
- net Dr2Enable: track 0.00 -> 77.7 mm
- net Dr2MS0: track 0.00 -> 74.8 mm
- net Dr2MS1: track 0.00 -> 70.5 mm
- net Dr2MS2: track 0.00 -> 69.7 mm, vias 0 -> 1
- net Dr2Step: track 0.00 -> 59.6 mm
- net Dr1Enable: track 0.00 -> 57.6 mm, vias 0 -> 1
- net Dr2Dir: track 0.00 -> 56.1 mm
- net Dr1MS2: track 0.00 -> 50.1 mm, vias 0 -> 1
- net Dr1MS0: track 0.00 -> 49.1 mm
- net Dr1Step: track 0.00 -> 48.5 mm
- net Dr1Dir: track 0.00 -> 48.0 mm
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- added copper zone on F.Cu, net +12V
Other:
- board outline added: 81.3 x 121.3 mm

Commit message: Merged with not-standart library
Parts:
- R13, R14: footprint SM0805_Opendous -> SM0805
- moved R13 2.54 mm to (315.6, 140.3), turned to 90 degrees
- moved R14 2.54 mm to (313.1, 140.3)
Routing:
- net AIN1: track 59.8 -> 42.9 mm
- net AIN3: track 64.3 -> 80.0 mm
- net VREF-: track 36.1 -> 38.0 mm
- net VREF+: track 24.7 -> 24.1 mm

Commit message: Continue drawing a PCB
Parts:
- added P1: POWER, bornier4, F.Cu at (340.4, 170.8)
- added X1: 8MHz, Crystal_7x5mm, F.Cu at (305.1, 133.5)
- R15, R16, R17, R18: footprint SM0805_Opendous -> SM0805; moved to B.Cu
- moved R15 178.7 mm to (374.6, 123.8)
- moved R16 164.3 mm to (368.3, 130.2)
- moved P13 146.0 mm to (370.2, 121.9), turned to 90 degrees
- moved P14 143.4 mm to (363.9, 128.9), turned to 90 degrees
- moved P22 143.3 mm to (304.8, 183.5), turned to 180 degrees
- moved P21 138.8 mm to (322.6, 183.5)
- moved P17 131.5 mm to (360.0, 111.3), turned to 0 degrees
- moved Q10 126.2 mm to (317.5, 177.2), turned to 270 degrees
- moved Q13 125.6 mm to (297.8, 171.4)
- moved R32 101.4 mm to (317.5, 172.1), turned to 270 degrees
- moved Q8 98.3 mm to (317.5, 168.3), turned to 0 degrees
- moved C28 95.8 mm to (317.5, 164.5), turned to 270 degrees
- moved R17 94.2 mm to (297.8, 134.6), turned to 270 degrees
- moved Q9 93.5 mm to (314.3, 169.5), turned to 0 degrees
- moved R30 93.0 mm to (315.6, 165.7), turned to 270 degrees
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Connections:
- net N-0000013 renamed PWM3OUT
- net N-0000067 renamed PWM1OUT
- P20 pad 3: N-0000063 (its old number) -> PWM2OUT
- P20 pad 4: N-0000063 (its old number) -> PWM2OUT
- P22 pad 3: N-0000019 (its old number) -> PWM4OUT
- P22 pad 4: N-0000019 (its old number) -> PWM4OUT
- Q13 pad 2: N-0000019 (its old number) -> PWM4OUT
- Q7 pad 2: N-0000063 (its old number) -> PWM2OUT
Routing:
- net +12V: track 15.5 -> 173.2 mm, vias 0 -> 5
- net Dr5Dir: track 0.00 -> 80.5 mm, vias 0 -> 2
- net Dr5Step: track 0.00 -> 78.5 mm, vias 0 -> 2
- net Dr5MS2: track 0.00 -> 68.3 mm, vias 0 -> 2
- net PWM2OUT: track 0.00 -> 67.7 mm, vias 0 -> 22
- net Dr5MS1: track 0.00 -> 66.5 mm, vias 0 -> 2
- net VCOM: track 244.7 -> 311.1 mm, vias 5 -> 13
- net Dr5MS0: track 0.00 -> 64.6 mm, vias 0 -> 2
- net Dr5Enable: track 0.00 -> 64.5 mm, vias 0 -> 1
- net Dr4Enable: track 0.00 -> 47.7 mm, vias 0 -> 1
- net Dr3Enable: track 0.00 -> 43.7 mm, vias 0 -> 1
- net PWM1OUT: track 28.2 -> 66.4 mm, vias 19 -> 22
- net IN3: track 0.00 -> 28.1 mm, vias 0 -> 1
- net N-0000063 (its old number): track 27.7 -> 0.00 mm, vias 19 -> 0
- net OUT5: track 0.00 -> 25.2 mm, vias 0 -> 1
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- added copper zone on B.Cu, net +12V
- added copper zone on B.Cu, net PWM1OUT
- added copper zone on F.Cu, net PWM1OUT
- added copper zone on B.Cu, net PWM2OUT
- added copper zone on F.Cu, net PWM2OUT
- added copper zone on F.Cu, net PWM3OUT
- added copper zone on F.Cu, net PWM4OUT
- removed copper zone on F.Cu, net +12V

Commit message: Update firmware
Parts:
- removed P2: BOOT, pin_socket_3
- removed R3, R4: 0,47, r_2512
- removed R8: 10k, SM0805
- added K1: UART, pin_socket_3, F.Cu at (331.2, 143.0)
- C1, C2, C3, D1, JP1, L1, R1, R2, R5, R6, U1: moved to B.Cu
- moved D1 87.3 mm to (302.3, 149.9), turned to 90 degrees
- moved C1 74.9 mm to (296.5, 165.7), turned to 180 degrees
- moved R2 74.8 mm to (295.9, 154.9), turned to 270 degrees
- moved L1 72.6 mm to (308.0, 150.7), turned to 270 degrees
- moved R1 71.9 mm to (292.1, 154.9), turned to 270 degrees
- moved C3 71.2 mm to (313.7, 151.8), turned to 90 degrees
- moved R15 70.3 mm to (306.1, 108.6)
- moved R16 70.1 mm to (301.6, 108.6), turned to 180 degrees
- moved P14 66.3 mm to (301.6, 106.0), turned to 0 degrees
- moved P13 64.2 mm to (308.0, 106.0), turned to 0 degrees
- moved P17 63.9 mm to (297.2, 99.7), turned to 90 degrees
- moved U1 61.1 mm to (297.2, 146.1)
- moved R5 56.3 mm to (293.4, 146.1), turned to 90 degrees
- moved C2 55.3 mm to (299.1, 141.0), turned to 180 degrees
- moved JP1 50.6 mm to (314.2, 124.7), turned to 135 degrees
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Connections:
- U2 pad 47: (no net) -> SlaveTX
- U2 pad 48: (no net) -> SlaveRX
Routing:
- net VCOM: track 311.1 -> 412.7 mm, vias 13 -> 35
- net PWM4: track 0.00 -> 59.1 mm, vias 0 -> 1
- net +12V: track 173.2 -> 222.8 mm
- net USBEN: track 0.00 -> 21.4 mm, vias 0 -> 2
- net IN2: track 0.00 -> 20.0 mm, vias 0 -> 1
- net SlaveTX: track 0.00 -> 20.0 mm
- net SlaveRX: track 0.00 -> 17.6 mm
- net IN1: track 0.00 -> 17.3 mm, vias 0 -> 1
- net N-0000021: track 0.00 -> 15.7 mm, vias 0 -> 2
- net N-0000070: track 0.00 -> 14.6 mm, vias 0 -> 2
- net N-0000071: track 0.00 -> 9.22 mm
- net BOOT0: track 0.00 -> 5.36 mm, vias 0 -> 1
- net VDD: track 148.6 -> 152.2 mm
- net OSC_OUT: track 2.28 -> 5.10 mm
- net N-0000022: track 0.00 -> 2.04 mm
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