File: schematics/rep_stm.sch (KiCad schematic (older format))
At the start: 1 part

Commit message: Drawing schematics
Parts:
- added C? (x11): 100n, ~, symbol C
- added C?: 4,7mF, ~, symbol CP
- added C? (x7): 10n, ~, symbol C
- added C? (x2): 1mF, ~, symbol CP
- added C? (x3): 22pF, ~, symbol C
- added C?: C, ~, symbol C
- added CON?: USB-MINI-B, symbol USB-MINI-B
- added IC? (x4): MOC3011M, DIP6, symbol MOC3011M
- added JP?: A2, ~, symbol JUMPER
- added JP?: A1, ~, symbol JUMPER
- added JP?: A0, ~, symbol JUMPER
- added JP?: BOOT0, ~, symbol JUMPER
- added K?: BOOT, symbol CONN_3
- added L? (x2): 10uH, ~, symbol INDUCTOR
- added P?: THERM1, symbol CONN_2
- added P?: THERM2, symbol CONN_2
- added P?: END1, symbol CONN_2
- added P?: END2, symbol CONN_2
- added P?: END3, symbol CONN_2
- added P?: END4, symbol CONN_2
- added P?: DIGITAL OUT, symbol CONN_7
- added P? (x5): POLOLU, symbol CONN_8X2
- added P?: DRIVE 1, symbol CONN_4
- added P?: DRIVE 2, symbol CONN_4
- added P?: DRIVE 3, symbol CONN_4
- added P?: DRIVE 4, symbol CONN_4
- added P?: DRIVE 5, symbol CONN_4
- added P?: PROG, symbol CONN_5
- added P?: ANALOG IN, symbol CONN_6
- added P?: DIGITAL INP, symbol CONN_7
- added P?: PWM 2, symbol CONN_4
- added P?: PWM 1, symbol CONN_4
- added P?: PWM 4, symbol CONN_4
- added P?: PWM 3, symbol CONN_4
- added P?: POWER, symbol CONN_4
- added Q? (x5): BC808-40, SOT-23, symbol BC808-40
- added Q? (x4): BC818-40, SOT-23, symbol BC818-40
- added Q? (x4): IRF540N, TO220, symbol IRF540N
- added R? (x15): 10k, ~, symbol R
- added R? (x2): 47k, ~, symbol R
- added R? (x2): 33R, ~, symbol R
- added R?: 1,5k, ~, symbol R
- added R?: 2,2k, ~, symbol R
- added R? (x4): 1k, ~, symbol R
- added R? (x4): 20R, ~, symbol R
- added U?: 24C512, symbol 24C512
- added X?: 8MHz, ~, symbol CRYSTAL_ACTIVE
Connections:
- net AIN10 is gone; now on net AIN6: U?.16 (ADC123_IN11/PC1)
- net AIN11 is gone; now on net IN7: U?.17 (ADC123_IN12/PC2)
- net AIN12 is gone; now on net IN8: U?.18 (ADC123_IN13/PC3)
- net AIN9 is gone; now on net AIN5: U?.15 (ADC123_IN10/PC0)
- net VREF+ is gone; now on net VAA: U?.21 (VREF+)
- net VREF- is gone; now on net AGND: U?.20 (VREF-)
- net AIN1: now also P?.2 (PM), R?.1
- net AIN2: now also P?.2
- net AIN3: now also U?.29 (SPI1_NSS/USART2_CK/DAC_OUT1/ADC12_IN4/PA4), P?.2 (PM), R?.1; no longer U?.25 (USART2_TX/TIM5_CH3/ADC123_IN2/TIM2_CH3/PA2)
- net AIN4: now also U?.30 (SPI1_SCK/DAC_OUT2/ADC12_IN5/PA5), P?.3; no longer U?.26 (USART2_RX/TIM5_CH4/ADC123_IN3/TIM2_CH4/PA3)
- net AIN5: now also P?.4; no longer U?.29 (SPI1_NSS/USART2_CK/DAC_OUT1/ADC12_IN4/PA4)
- net AIN6: now also P?.5; no longer U?.30 (SPI1_SCK/DAC_OUT2/ADC12_IN5/PA5)
- net BOOT0: now also JP?.2, K?.1 (P1), R?.2
- net DM: now also C?.1, R?.1
- net Dr1Dir: now also P?.15
- net Dr1MS0: now also P?.3
- net Dr1MS1: now also P?.5
- net Dr1MS2: now also K?.2 (PM), P?.7
- net Dr1Step: now also P?.13
- net Dr2Dir: now also P?.15
- net Dr2MS0: now also P?.3
- net Dr2MS1: now also P?.5
- net Dr2MS2: now also P?.7
- net Dr2Step: now also P?.13
- net Dr3Dir: now also P?.15
- net Dr3MS0: now also P?.3
- net Dr3MS1: now also P?.5
- net Dr3MS2: now also P?.7
- net Dr3Step: now also P?.13
- net Dr4Dir: now also P?.15
- net Dr4MS0: now also P?.3
- net Dr4MS1: now also P?.5
- net Dr4Step: now also P?.13
- net Dr5Dir: now also P?.15
- net Dr5MS0: now also P?.3
- net Dr5MS1: now also P?.5
- net Dr5MS2: now also P?.7
- net Dr5Step: now also P?.13
- net I2C_SCL: now also U?.6 (SCL)
- net I2C_SDA: now also U?.5 (SDA)
- net IN1: now also P?.1 (P1), R?.2
- net IN2: now also P?.1 (P1), R?.2
- net IN3: now also P?.1 (P1), R?.2
- net IN4: now also P?.1 (P1), R?.2
- net IN5: now also P?.1 (P1)
- net IN6: now also P?.2 (P2)
- net IN7: now also P?.3 (P3)
- net IN8: now also P?.4 (P4)
- net NRST: now also C?.1, P?.1, R?.2
- net OSC_OUT: now also C?.1, X?.3 (OUT)
- net OUT1: now also P?.1 (P1)
- net OUT2: now also P?.2 (P2)
- net OUT3: now also P?.3 (P3)
- net OUT4: now also P?.4 (P4)
- net OUT5: now also P?.5 (P5)
- net OUT6: now also P?.6 (P6)
- net PWM1: now also IC?.1
- net PWM2: now also IC?.1
- net PWM3: now also IC?.1
- net PWM4: now also IC?.1
- net SWCLK: now also P?.3
- net SWDIO: now also P?.2
- net VSS: now reaches U?.10 (VSS)
- net VSS: now also U?.27 (VSS), U?.49 (VSS), U?.74 (VSS), U?.99 (VSS), C?.1, C?.1, C?.1, C?.1, C?.1, C?.2, C?.2, C?.2, C?.2, C?.2, C?.2, C?.2, C?.2, C?.2, C?.2, C?.2, C?.2, C?.2, C?.2, CON?.5 (GND), CON?.6 (SHELL1), CON?.7 (SHELL2), CON?.8 (SHELL3), CON?.9 (SHELL4), IC?.2, IC?.2, IC?.2, IC?.2, JP?.1, JP?.1, JP?.1, JP?.1, K?.3 (P3), L?.1, P?.16, P?.16, P?.16, P?.16, P?.16, P?.2 (PM), P?.2 (PM), P?.2 (PM), P?.2 (PM), P?.4, P?.7 (P7), P?.7 (P7), U?.4 (GND), X?.2 (GND)
- net VDD: now reaches U?.100 (VDD)
- net VDD: now also U?.11 (VDD), U?.28 (VDD), U?.50 (VDD), U?.75 (VDD), C?.1, C?.1, C?.1, C?.1, C?.1, C?.1, C?.1, C?.1, C?.1, C?.1, C?.2, C?.2, C?.2, C?.2, C?.2, L?.1, P?.14, P?.14, P?.14, P?.14, P?.14, P?.5, Q?.2 (E), R?.1, R?.1, R?.1, R?.1, R?.1, R?.1, R?.1, R?.1, R?.1, R?.1, R?.1, U?.8 (VCC), X?.4 (VDD)
- net AGND: now reaches U?.19 (VSSA)
- net AGND: now also C?.2, C?.2, L?.2, P?.1, P?.6, R?.2, R?.2
- net VAA: now reaches U?.22 (VDDA)
- net VAA: now also C?.1, C?.1, L?.2, P?.1 (P1), P?.1 (P1)
- net USBEN: now reaches U?.53 (SPI2_MISO/TIM1_CH2N/USART3_RTS/PB14)
- net USBEN: now also R?.1
- net AIN7: no longer names the net of U?.31 (SPI1_MISO/TIM8_BKIN/ADC12_IN6/TIM3_CH1/PA6)
- net AIN8: no longer names the net of U?.32 (SPI1_MOSI/TIM8_CH1N/ADC12_IN7/TIM3_CH2/PA7)
- new net: JP?.2, R?.2, U?.1 (A0)
- new net: JP?.2, R?.2, U?.2 (A1)
- new net: JP?.2, R?.2, U?.3 (A2)
- new net: R?.2, U?.7 (WP)
- new net: P?.10, P?.3 (P3) (x5)
- new net: P?.11, P?.9 (x5)
- new net: P?.12, P?.4 (P4) (x5)
- new net: P?.1 (P1), P?.6 (x5)
- new net: P?.2 (P2), P?.8 (x5)
- new net: CON?.2 (D-), R?.2
- new net: CON?.3 (D+), R?.2
- new net: C?.1, R?.1, R?.2
- new net: Q?.3 (C), R?.1
- new net: Q?.1 (B), R?.2, R?.2
- new net: Q?.1 (B), Q?.1 (B), R?.2 (x4)
- new net: Q?.2 (E), Q?.2 (E), R?.1 (x4)
- new net: IC?.6, R?.1, R?.1 (x4)
- new net: Q?.1 (G), R?.2 (x4)
- new net: P?.3 (P3), P?.4 (P4), Q?.2 (D) (x4)
- new net +12V: C?.1, C?.1, C?.1, C?.1, P?.1 (P1), P?.1 (P1), P?.1 (P1), P?.1 (P1), P?.2, P?.2, P?.2, P?.2, P?.2, P?.2 (P2), P?.2 (P2), P?.2 (P2), P?.2 (P2), P?.3 (P3), P?.4 (P4), Q?.3 (C), Q?.3 (C), Q?.3 (C), Q?.3 (C), R?.2, R?.2, R?.2, R?.2
- new net Dr4MS2: P?.7
- new net IN10: P?.6 (P6), U?.26 (USART2_RX/TIM5_CH4/ADC123_IN3/TIM2_CH4/PA3)
- new net IN9: P?.5 (P5), U?.25 (USART2_TX/TIM5_CH3/ADC123_IN2/TIM2_CH3/PA2)
- new net VCOM: C?.2, C?.2, C?.2, C?.2, IC?.4, IC?.4, IC?.4, IC?.4, P?.1 (P1), P?.2 (P2), P?.4, P?.4, P?.4, P?.4, P?.4, Q?.3 (C), Q?.3 (C), Q?.3 (C), Q?.3 (C), Q?.3 (S), Q?.3 (S), Q?.3 (S), Q?.3 (S)

Commit message: Unfinished drawing...
Parts:
- added C1: 100u, ~, symbol CP
- added C2: 150pF, ~, symbol C
- added C3: 47uF, ~, symbol CP
- added D1: 1N5819, ~, symbol DIODESCH
- added L1: 22uH, ~, symbol INDUCTOR
- added R1, R2, R3, R4: 0,47, ~, symbol R
- added R5: 1,2k, ~, symbol R
- added R6: 2k, ~, symbol R
- added U1: MC34063, symbol MC34063
- gave numbers to parts that had none: 86
Connections:
- net VSS is gone; now on net VCOM: C10.2, C11.2, C14.2, C15.2, C16.2, C17.2, C18.1, C19.1, C20.1, C21.1, C22.1, C23.2, C24.2, C4.2, C5.2, C6.2, C7.2, C8.2, C9.2, IC1.2, IC2.2, IC3.2, IC4.2, JP1.1, JP2.1, JP3.1, JP4.1, L3.1, M1.16, M2.16, M3.16, M4.16, M5.16, P12.2 (PM), P13.2 (PM), P14.2 (PM), P15.2 (PM), P16.7 (P7), P2.3 (P3), P3.4, P9.7 (P7), U2.10 (VSS), U2.27 (VSS), U2.49 (VSS), U2.74 (VSS), U2.99 (VSS), U3.4 (GND), X1.2 (GND), p17.5 (GND), p17.6 (SHELL1), p17.7 (SHELL2), p17.8 (SHELL3), p17.9 (SHELL4)
- net +12V: now also C1.1, R1.1, R2.1, R3.1, R4.1, U1.6 (VCC)
- net DP: now also C24.1, R21.2, R23.1
- net VCOM: now also C1.2, C2.2, C3.2, D1.1 (A), R5.2, U1.4 (GND)
- net VDD: now also C3.1, L1.2, R6.2
- new net: R1.2, R2.2, R3.2, R4.2, U1.1 (Sw_Coll), U1.7 (I_Sense), U1.8 (Drv_Coll)
- new net: D1.2 (K), L1.1, U1.2 (Sw_Emit)
- new net: C2.1, U1.3 (Tim_Cap)
- new net: R5.1, R6.1, U1.5 (V_Sense)
Other:
- moved on the sheet: P1

Commit message: Fixed schematics
Parts:
- removed C18, C19, C20, C21, C22: 100n, ~, symbol C
- added C18, C19, C20, C21, C22: 100uFx25V, ~, symbol CP
- added C29, C30, C31, C32, C33, C34: 10uF, ~, symbol CP
- added R36, R37, R38, R39: 47k, ~, symbol R
- C11, C13: value 1mF -> 1uF
- C16: value C -> 100n
- C9: value 4,7mF -> 4,7uF
- Q10, Q13, Q4, Q7: value IRF540N -> IRF1404S
- gave numbers to parts that had none: 20
- renumbered P12 to P13, P13 to P14, P14 to P15, P15 to P16, P16 to P17, p17 to P18
Connections:
- net AGND: now also R36.2, R37.2, R38.2, R39.2; no longer P12.1
- net AIN1: now also C29.2
- net AIN2: now also C31.2, R36.1
- net AIN3: now also C30.2
- net AIN4: now also C32.2, R37.1
- net AIN5: now also C33.2, R38.1
- net AIN6: now also C34.2, R39.1
- net VAA: now also P12.1, C29.1, C30.1, C31.1, C32.1, C33.1, C34.1
- net VCOM: now also C18.1, C19.1, C20.1, C21.1, C22.1
- net VDD: now also C18.2, C19.2, C20.2, C21.2, C22.2
- net Dr1Enable: now reaches U2.43 (PE12/FSMC_D9)
- net Dr1Enable: now also M1.1
- net Dr2Enable: now reaches U2.44 (PE13/FSMC_D10)
- net Dr2Enable: now also M2.1
- net Dr3Enable: now reaches U2.45 (PE14/FSMC_D11)
- net Dr3Enable: now also M3.1
- net Dr4Enable: now reaches U2.46 (PE15/FSMC_D12)
- net Dr4Enable: now also M4.1
- net Dr5Enable: now reaches U2.51 (SPI2_NSS/I2S2_WS/I2C2_SMBA/USART3_CK/TIM1_BKIN/PB12)
- net Dr5Enable: now also M5.1
Other:
- moved on the sheet: M2, M3, P10, P12, P5, P6, R13, R14

Commit message: Start drawing a PCB
Parts:
- removed M1, M2, M3, M4, M5: POLOLU, symbol CONN_8X2
- added C35, C36, C37, C38, C39: 100n, ~, symbol C
- added U4, U5, U6, U7, U8: POLOLU_A4988, symbol POLOLU_A4988
Connections:
- net +12V: now also C18.2, C19.2, C20.2, C21.2, C22.2, U4.8 (VMOT), U5.8 (VMOT), U6.8 (VMOT), U7.8 (VMOT), U8.8 (VMOT)
- net Dr1Dir: now also U4.16 (DIR)
- net Dr1Enable: now also U4.9 (EN)
- net Dr1MS0: now also U4.10 (MS1)
- net Dr1MS1: now also U4.11 (MS2)
- net Dr1MS2: now also U4.12 (MS3)
- net Dr1Step: now also U4.15 (STEP)
- net Dr2Dir: now also U5.16 (DIR)
- net Dr2Enable: now also U5.9 (EN)
- net Dr2MS0: now also U5.10 (MS1)
- net Dr2MS1: now also U5.11 (MS2)
- net Dr2MS2: now also U5.12 (MS3)
- net Dr2Step: now also U5.15 (STEP)
- net Dr3Dir: now also U6.16 (DIR)
- net Dr3Enable: now also U6.9 (EN)
- net Dr3MS0: now also U6.10 (MS1)
- net Dr3MS1: now also U6.11 (MS2)
- net Dr3MS2: now also U6.12 (MS3)
- net Dr3Step: now also U6.15 (STEP)
- net Dr4Dir: now also U7.16 (DIR)
- net Dr4Enable: now also U7.9 (EN)
- net Dr4MS0: now also U7.10 (MS1)
- net Dr4MS1: now also U7.11 (MS2)
- net Dr4MS2: now also U7.12 (MS3)
- net Dr4Step: now also U7.15 (STEP)
- net Dr5Dir: now also U8.16 (DIR)
- net Dr5Enable: now also U8.9 (EN)
- net Dr5MS0: now also U8.10 (MS1)
- net Dr5MS1: now also U8.11 (MS2)
- net Dr5MS2: now also U8.12 (MS3)
- net Dr5Step: now also U8.15 (STEP)
- net VCOM: now also C35.1, C36.1, C37.1, C38.1, C39.1, U4.1 (GND), U4.7 (GND), U5.1 (GND), U5.7 (GND), U6.1 (GND), U6.7 (GND), U7.1 (GND), U7.7 (GND), U8.1 (GND), U8.7 (GND)
- net VDD: now also C35.2, C36.2, C37.2, C38.2, C39.2, U4.2 (VDD), U5.2 (VDD), U6.2 (VDD), U7.2 (VDD), U8.2 (VDD); no longer C18.2, C19.2, C20.2, C21.2, C22.2
- net at P4.3 (P3): now also U4.4 (1A)
- net at P4.4 (P4): now also U4.3 (IB)
- net at P4.1 (P1): now also U4.6 (2B)
- net at P4.2 (P2): now also U4.5 (2A)
- net at P5.3 (P3): now also U5.4 (1A)
- net at P5.4 (P4): now also U5.3 (IB)
- net at P5.1 (P1): now also U5.6 (2B)
- net at P5.2 (P2): now also U5.5 (2A)
- net at P6.3 (P3): now also U6.4 (1A)
- net at P6.4 (P4): now also U6.3 (IB)
- net at P6.1 (P1): now also U6.6 (2B)
- net at P6.2 (P2): now also U6.5 (2A)
- net at P7.3 (P3): now also U7.4 (1A)
- net at P7.4 (P4): now also U7.3 (IB)
- net at P7.1 (P1): now also U7.6 (2B)
- net at P7.2 (P2): now also U7.5 (2A)
- net at P8.3 (P3): now also U8.4 (1A)
- net at P8.4 (P4): now also U8.3 (IB)
- net at P8.1 (P1): now also U8.6 (2B)
- net at P8.2 (P2): now also U8.5 (2A)
- new net: U4.13 (RST), U4.14 (SLP)
- new net: U5.13 (RST), U5.14 (SLP)
- new net: U6.13 (RST), U6.14 (SLP)
- new net: U7.13 (RST), U7.14 (SLP)
- new net: U8.13 (RST), U8.14 (SLP)
Other:
- moved on the sheet: C18, C19, C20, C21, C22, C29, C30, P10, P11, P4, P5, P6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

Commit message: Continue drawing a PCB
Connections:
- net PWM1OUT: now also P19.3 (P3), P19.4 (P4), Q4.2 (D)
- net PWM2OUT: now also P20.3 (P3), P20.4 (P4), Q7.2 (D)
- net PWM3OUT: now also P21.3 (P3), P21.4 (P4), Q10.2 (D)
- net PWM4OUT: now also P22.3 (P3), P22.4 (P4), Q13.2 (D)
Changed lines of the file:
@@
 Sheet 1 1
 Title "RepRap STM32 Ver."
-Date "10 nov 2014"
+Date "11 nov 2014"
 Rev ""
 Comp ""
@@
 	11750 2300 11750 2150
 Wire Wire Line
-	11750 2150 11800 2150
+	11700 2150 11800 2150
 Wire Wire Line
 	11800 2250 11750 2250
@@
 	11750 1050 11750 900
 Wire Wire Line
-	11750 900  11800 900
+	11700 900  11800 900
 Wire Wire Line
 	11800 1000 11750 1000
@@
 	15350 2350 15350 2200
 Wire Wire Line
-	15350 2200 15400 2200
+	15300 2200 15400 2200
 Wire Wire Line
 	15400 2300 15350 2300
@@
 	15350 1100 15350 950
 Wire Wire Line
-	15350 950  15400 950
+	15300 950  15400 950
 Wire Wire Line
 	15400 1050 15350 1050
@@
 	0    1    1    0
 $EndComp
-Text Label 11300 850  0    60   ~ 0
+Text GLabel 11700 900  0    60   Input ~ 0
 PWM1OUT
-Text Label 11300 2100 0    60   ~ 0
+Text GLabel 11700 2150 0    60   Input ~ 0
 PWM2OUT
-Text Label 14950 850  0    60   ~ 0
+Text GLabel 15300 950  0    60   Input ~ 0
 PWM3OUT
-Text Label 14850 2150 0    60   ~ 0
+Text GLabel 15300 2200 0    60   Input ~ 0
 PWM4OUT
+Connection ~ 15350 2200
+Connection ~ 15350 950
+Connection ~ 11750 2150
+Connection ~ 11750 900
 $EndSCHEMATC

Commit message: Update firmware
Parts:
- added K1: UART, ~, symbol CONN_3
Connections:
- net SlaveRX: now also K1.2 (PM)
- net SlaveTX: now also K1.1 (P1)
- net VCOM: now also K1.3 (P3)
Changed lines of the file:
@@
 Sheet 1 1
 Title "RepRap STM32 Ver."
-Date "11 nov 2014"
+Date "12 nov 2014"
 Rev ""
 Comp ""
@@
 $EndComp
 $Comp
-L VCOM #PWR48
+L VCOM #PWR49
 U 1 1 545FCEDD
 P 6850 3450
-F 0 "#PWR48" H 6850 3650 40  0001 C CNN
+F 0 "#PWR49" H 6850 3650 40  0001 C CNN
 F 1 "VCOM" H 6850 3600 40  0000 C CNN
 F 2 "" H 6850 3450 60  0000 C CNN
@@
 $EndComp
 $Comp
-L VCOM #PWR49
+L VCOM #PWR50
 U 1 1 545FD552
 P 9050 3450
-F 0 "#PWR49" H 9050 3650 40  0001 C CNN
+F 0 "#PWR50" H 9050 3650 40  0001 C CNN
 F 1 "VCOM" H 9050 3600 40  0000 C CNN
 F 2 "" H 9050 3450 60  0000 C CNN
@@
 $EndComp
 $Comp
-L VCOM #PWR50
+L VCOM #PWR51
 U 1 1 545FD720
 P 11250 3450
-F 0 "#PWR50" H 11250 3650 40  0001 C CNN
+F 0 "#PWR51" H 11250 3650 40  0001 C CNN
 F 1 "VCOM" H 11250 3600 40  0000 C CNN
 F 2 "" H 11250 3450 60  0000 C CNN
@@
 $EndComp
 $Comp
-L VCOM #PWR72
+L VCOM #PWR73
 U 1 1 545FD75E
 P 6650 4800
-F 0 "#PWR72" H 6650 5000 40  0001 C CNN
+F 0 "#PWR73" H 6650 5000 40  0001 C CNN
 F 1 "VCOM" H 6650 4950 40  0000 C CNN
 F 2 "" H 6650 4800 60  0000 C CNN
@@
 $EndComp
 $Comp
-L VCOM #PWR73
+L VCOM #PWR74
 U 1 1 545FDABD
 P 8750 4800
-F 0 "#PWR73" H 8750 5000 40  0001 C CNN
+F 0 "#PWR74" H 8750 5000 40  0001 C CNN
 F 1 "VCOM" H 8750 4950 40  0000 C CNN
 F 2 "" H 8750 4800 60  0000 C CNN
@@
 $EndComp
 $Comp
-L VCOM #PWR43
+L VCOM #PWR44
 U 1 1 546016E1
 P 10900 3000
-F 0 "#PWR43" H 10900 3200 40  0001 C CNN
+F 0 "#PWR44" H 10900 3200 40  0001 C CNN
 F 1 "VCOM" H 10900 3150 40  0000 C CNN
 F 2 "" H 10900 3000 60  0000 C CNN
@@
 $EndComp
 $Comp
-L VCOM #PWR44
+L VCOM #PWR45
 U 1 1 5460270C
 P 14500 3050
-F 0 "#PWR44" H 14500 3250 40  0001 C CNN
+F 0 "#PWR45" H 14500 3250 40  0001 C CNN
 F 1 "VCOM" H 14500 3200 40  0000 C CNN
 F 2 "" H 14500 3050 60  0000 C CNN
@@
 $EndComp
 $Comp
-L VCOM #PWR138
+L VCOM #PWR139
 U 1 1 54603026
 P 12750 7450
-F 0 "#PWR138" H 12750 7650 40  0001 C CNN
+F 0 "#PWR139" H 12750 7650 40  0001 C CNN
 F 1 "VCOM" H 12750 7600 40  0000 C CNN
 F 2 "" H 12750 7450 60  0000 C CNN
@@
 $EndComp
 $Comp
-L VCOM #PWR113
+L VCOM #PWR114
 U 1 1 545FD48B
 P 12450 6600
-F 0 "#PWR113" H 12450 6800 40  0001 C CNN
+F 0 "#PWR114" H 12450 6800 40  0001 C CNN
 F 1 "VCOM" H 12450 6750 40  0000 C CNN
 F 2 "" H 12450 6600 60  0000 C CNN
@@
 $EndComp
 $Comp
-L VCOM #PWR128
+L VCOM #PWR129
 U 1 1 545FD491
 P 14000 7350
-F 0 "#PWR128" H 14000 7550 40  0001 C CNN
+F 0 "#PWR129" H 14000 7550 40  0001 C CNN
 F 1 "VCOM" H 14000 7500 40  0000 C CNN
 F 2 "" H 14000 7350 60  0000 C CNN
@@
 $EndComp
 $Comp
-L VCOM #PWR141
+L VCOM #PWR142
 U 1 1 545FDC56
 P 15000 7600
-F 0 "#PWR141" H 15000 7800 40  0001 C CNN
+F 0 "#PWR142" H 15000 7800 40  0001 C CNN
 F 1 "VCOM" H 15000 7750 40  0000 C CNN
 F 2 "" H 15000 7600 60  0000 C CNN
@@
 $EndComp
 $Comp
-L VCOM #PWR109
+L VCOM #PWR110
 U 1 1 545FDEB8
 P 15050 6450
-F 0 "#PWR109" H 15050 6650 40  0001 C CNN
+F 0 "#PWR110" H 15050 6650 40  0001 C CNN
 F 1 "VCOM" H 15050 6600 40  0000 C CNN
 F 2 "" H 15050 6450 60  0000 C CNN
@@
 $EndComp
 $Comp
-L VCOM #PWR140
+L VCOM #PWR141
 U 1 1 545FE555
 P 15750 7500
-F 0 "#PWR140" H 15750 7700 40  0001 C CNN
+F 0 "#PWR141" H 15750 7700 40  0001 C CNN
 F 1 "VCOM" H 15750 7650 40  0000 C CNN
 F 2 "" H 15750 7500 60  0000 C CNN
@@
 $EndComp
 $Comp
-L VCOM #PWR137
+L VCOM #PWR138
 U 1 1 545FE8B9
 P 13000 7400
-F 0 "#PWR137" H 13000 7600 40  0001 C CNN
+F 0 "#PWR138" H 13000 7600 40  0001 C CNN
 F 1 "VCOM" H 13000 7550 40  0000 C CNN
 F 2 "" H 13000 7400 60  0000 C CNN
@@
 $EndComp
 $Comp
-L VCOM #PWR105
+L VCOM #PWR106
 U 1 1 545FEC0F
 P 15650 6350
-F 0 "#PWR105" H 15650 6550 40  0001 C CNN
+F 0 "#PWR106" H 15650 6550 40  0001 C CNN
 F 1 "VCOM" H 15650 6500 40  0000 C CNN
 F 2 "" H 15650 6350 60  0000 C CNN
@@
 Connection ~ 11750 2150
 Connection ~ 11750 900
+Text GLabel 7550 2750 0    60   Input ~ 0
+SlaveTX
+Text GLabel 7550 2850 0    60   Input ~ 0
+SlaveRX
+$Comp
+L CONN_3 K1
+U 1 1 5462F7A6
+P 7900 2850
+F 0 "K1" V 7850 2850 50  0000 C CNN
+F 1 "UART" V 7950 2850 40  0000 C CNN
+F 2 "~" H 7900 2850 60  0000 C CNN
+F 3 "~" H 7900 2850 60  0000 C CNN
+	1    7900 2850
+	1    0    0    -1
+$EndComp
+$Comp
+L VSS #PWR0114
+U 1 1 5462F7B3
+P 7550 2950
+F 0 "#PWR0114" H 7550 2950 30  0001 C CNN
+F 1 "VSS" H 7550 2880 30  0000 C CNN
+F 2 "" H 7550 2950 60  0000 C CNN
+F 3 "" H 7550 2950 60  0000 C CNN
+	1    7550 2950
+	0    1    1    0
+$EndComp
 $EndSCHEMATC
